File: HW/ESR-Meter/User_Interface.kicad_sch (KiCad schematic)
At the start: 0 parts

Commit message: HW Started
Other:
- added sheet Buttons (Buttons.kicad_sch)
- added sheet Display (Display.kicad_sch)
Changed lines of the file:
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@@
 (kicad_sch (version 20211123) (generator eeschema)
   (paper "A4")
+  (sheet (at 104.521 69.088) (size 32.766 33.528) (fields_autoplaced)
+    (stroke (width 0.1524) (type solid) (color 0 0 0 0))
+    (fill (color 0 0 0 0.0000))
+    (property "Sheet name" "Display" (id 0) (at 104.521 68.3764 0)
+      (effects (font (size 1.27 1.27)) (justify left bottom))
+    )
+    (property "Sheet file" "Display.kicad_sch" (id 1) (at 104.521 103.2006 0)
+      (effects (font (size 1.27 1.27)) (justify left top))
+    )
+  )
+  (sheet (at 104.521 28.956) (size 33.02 26.035) (fields_autoplaced)
+    (stroke (width 0.1524) (type solid) (color 0 0 0 0))
+    (fill (color 0 0 0 0.0000))
+    (property "Sheet name" "Buttons" (id 0) (at 104.521 28.2444 0)
+      (effects (font (size 1.27 1.27)) (justify left bottom))
+    )
+    (property "Sheet file" "Buttons.kicad_sch" (id 1) (at 104.521 55.5756 0)
+      (effects (font (size 1.27 1.27)) (justify left top))
+    )
+  )
 )
