File: HW/ESR-Meter/Display Controller.kicad_sch (KiCad schematic)
At the start: 0 parts

Commit message: Display controller
Parts:
- added C1101: (no value), symbol Device:C_Small
- added IC1101: (no value), symbol 74xx:74HC595
- added R1101, R1102, R1103, R1104, R1105, R1106, R1107, R1108, R1109, R1110, R1111, R1112: (no value), symbol Device:R_Small
Connections:
- net DISP_CLK: now also R1102.1
- net DISP_DATA: now also R1101.1
- net DISP_STRB: now also R1104.1
- new net: IC1101.5 (QF), R1110.1
- new net: IC1101.3 (QD), R1108.1
- new net: IC1101.12 (RCLK), R1104.2
- new net: IC1101.2 (QC), R1107.1
- new net: IC1101.7 (QH), R1112.1
- new net: IC1101.11 (SRCLK), R1102.2
- new net: IC1101.15 (QA), R1105.1
- new net: IC1101.4 (QE), R1109.1
- new net: IC1101.6 (QG), R1111.1
- new net: IC1101.14 (SER), R1101.2
- new net: IC1101.10 (~{SRCLR}), R1103.2
- new net: IC1101.1 (QB), R1106.1
- new net A: R1105.2
- new net B: R1106.2
- new net C: R1107.2
- new net D: R1108.2
- new net DISP_RST: R1103.1
- new net DP: R1112.2
- new net E: R1109.2
- new net F: R1110.2
- new net G: R1111.2
- new net GND: C1101.2, IC1101.13 (~{OE}), IC1101.8 (GND)
- new net VCC: C1101.1, IC1101.16 (VCC)
- no-connect marks 0 -> 1
