File: HW/ESR-Meter/ESR-Meter.kicad_sch (KiCad schematic)
At the start: 0 parts

Commit message: HW Started
Other:
- added sheet Current Generator (Current Generator.kicad_sch)
- added sheet PSU (PSU.kicad_sch)
- added sheet Reference (Reference.kicad_sch)
- added sheet Signal Amplifier (Signal amplifier.kicad_sch)
Changed lines of the file:
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@@
 (kicad_sch (version 20211123) (generator eeschema)
   (paper "A4")
-  (sheet (at 118.872 64.262) (size 22.987 33.274) (fields_autoplaced)
+  (sheet (at 71.247 67.31) (size 19.812 10.414) (fields_autoplaced)
     (stroke (width 0.1524) (type solid) (color 0 0 0 0))
     (fill (color 0 0 0 0.0000))
-    (property "Sheet name" "MCU" (id 0) (at 118.872 63.5504 0)
+    (property "Sheet name" "Current Generator" (id 0) (at 71.247 66.5984 0)
       (effects (font (size 1.27 1.27)) (justify left bottom))
     )
-    (property "Sheet file" "MCU.kicad_sch" (id 1) (at 118.872 98.1206 0)
+    (property "Sheet file" "Current Generator.kicad_sch" (id 1) (at 71.247 78.3086 0)
       (effects (font (size 1.27 1.27)) (justify left top))
     )
   )
-  (sheet (at 165.481 80.772) (size 14.732 10.414) (fields_autoplaced)
+  (sheet (at 105.664 50.546) (size 25.654 42.164) (fields_autoplaced)
     (stroke (width 0.1524) (type solid) (color 0 0 0 0))
     (fill (color 0 0 0 0.0000))
-    (property "Sheet name" "User Interface" (id 0) (at 165.481 80.0604 0)
+    (property "Sheet name" "MCU" (id 0) (at 105.664 49.8344 0)
       (effects (font (size 1.27 1.27)) (justify left bottom))
     )
-    (property "Sheet file" "User_Interface.kicad_sch" (id 1) (at 165.481 91.7706 0)
+    (property "Sheet file" "MCU.kicad_sch" (id 1) (at 105.664 93.2946 0)
+      (effects (font (size 1.27 1.27)) (justify left top))
+    )
+  )
+  (sheet (at 138.43 67.437) (size 22.733 25.273) (fields_autoplaced)
+    (stroke (width 0.1524) (type solid) (color 0 0 0 0))
+    (fill (color 0 0 0 0.0000))
+    (property "Sheet name" "User Interface" (id 0) (at 138.43 66.7254 0)
+      (effects (font (size 1.27 1.27)) (justify left bottom))
+    )
+    (property "Sheet file" "User_Interface.kicad_sch" (id 1) (at 138.43 93.2946 0)
+      (effects (font (size 1.27 1.27)) (justify left top))
+    )
+  )
+  (sheet (at 71.374 83.566) (size 19.304 8.763) (fields_autoplaced)
+    (stroke (width 0.1524) (type solid) (color 0 0 0 0))
+    (fill (color 0 0 0 0.0000))
+    (property "Sheet name" "Signal Amplifier" (id 0) (at 71.374 82.8544 0)
+      (effects (font (size 1.27 1.27)) (justify left bottom))
+    )
+    (property "Sheet file" "Signal amplifier.kicad_sch" (id 1) (at 71.374 92.9136 0)
+      (effects (font (size 1.27 1.27)) (justify left top))
+    )
+  )
+  (sheet (at 71.12 50.546) (size 20.193 11.049) (fields_autoplaced)
+    (stroke (width 0.1524) (type solid) (color 0 0 0 0))
+    (fill (color 0 0 0 0.0000))
+    (property "Sheet name" "Reference" (id 0) (at 71.12 49.8344 0)
+      (effects (font (size 1.27 1.27)) (justify left bottom))
+    )
+    (property "Sheet file" "Reference.kicad_sch" (id 1) (at 71.12 62.1796 0)
+      (effects (font (size 1.27 1.27)) (justify left top))
+    )
+  )
+  (sheet (at 138.43 50.673) (size 22.86 11.049) (fields_autoplaced)
+    (stroke (width 0.1524) (type solid) (color 0 0 0 0))
+    (fill (color 0 0 0 0.0000))
+    (property "Sheet name" "PSU" (id 0) (at 138.43 49.9614 0)
+      (effects (font (size 1.27 1.27)) (justify left bottom))
+    )
+    (property "Sheet file" "PSU.kicad_sch" (id 1) (at 138.43 62.3066 0)
       (effects (font (size 1.27 1.27)) (justify left top))
     )
@@
     (path "/609b9e1b-4e3b-42b7-ac76-a62ec4d0e7c7" (page "2"))
     (path "/6d646c30-feab-4e3e-adf0-5427b73b5f08" (page "3"))
+    (path "/d4ef5db0-5fba-4fcd-ab64-2ef2646c5c6d" (page "4"))
+    (path "/a09cb1c4-cc63-49c7-a35f-4b80c3ba2217" (page "5"))
+    (path "/337d1242-91ab-4446-8b9e-7609c6a49e3c" (page "6"))
+    (path "/7308e13a-4809-4e8e-af65-9905819aa376" (page "7"))
+    (path "/6d646c30-feab-4e3e-adf0-5427b73b5f08/fa96c103-a249-4d74-a8f7-f53b2f60fbfe" (page "8"))
+    (path "/6d646c30-feab-4e3e-adf0-5427b73b5f08/dc23c328-65de-43fb-a914-8938066176bf" (page "9"))
+    (path "/6d646c30-feab-4e3e-adf0-5427b73b5f08/dc23c328-65de-43fb-a914-8938066176bf/3594873d-d94b-4e9e-b5b1-5b1442595696" (page "10"))
+    (path "/6d646c30-feab-4e3e-adf0-5427b73b5f08/dc23c328-65de-43fb-a914-8938066176bf/d56fcef4-f1b8-4d2f-930b-7fbea51f96ea" (page "11"))
   )
 )
